Commit message: Add files via upload

File: hexapod_description/urdf/hexapod_description.urdf (robot description, URDF)
Before this commit: robot hexapod_description, 19 links, 18 joints
Links:
- link 1A_link: mass 0.0263699506965405 -> 0.0263699506965419
- link 1B_link: mass 0.0393326464255885 -> 0.0393326464255896
- link 1C_link: mass 0.0544820458081966 -> 0.0544820458081967
- link 2C_link: mass 0.0544820458081965 -> 0.0544820458081966
- link 3A_link: mass 0.0263699508271743 -> 0.0263699508271746
- link 3B_link: mass 0.039332646556227 -> 0.0393326465562273
- link 3C_link: mass 0.0544820458081966 -> 0.0544820458081965
- link 4A_link: mass 0.0263699506960539 -> 0.0263699506960721
- link 4B_link: mass 0.0393326464251206 -> 0.0393326464251387
- link 4C_link: mass 0.0544820458081967 -> 0.0544820458081966
- link 5A_link: mass 0.026369950689219 -> 0.0263699506893305
- link 5B_link: mass 0.0393326465545752 -> 0.0393326465545736
- link 5C_link: mass 0.0544820458081967 -> 0.0544820458081965
- link 6A_link: mass 0.0263699508281299 -> 0.0263699508281301
- link 6B_link: mass 0.0393326465581174 -> 0.0393326465581178
Joints:
- joint 1A_joint: axis 0 0 1 -> 0 0 0.999999999991391; origin xyz=-0.25962 -1.0213 -0.26955 rpy=1.5708 0 0 -> xyz=-0.0667468494517693 -0.106777799204074 0.0316495863697956 rpy=0 0 -0.541135476375613
- joint 1B_joint: axis 0.00033224 0.00037237 -1 -> -0.99634 0.085496 0; origin xyz=-0.0063327 -0.075236 -0.003549 rpy=1.5708 0.84229 1.4857 -> xyz=-0.0076049 -0.075127 -0.002699 rpy=0 0 0
- joint 1C_joint: axis 0 0 0 -> -0.99634 0.085496 0; origin xyz=-0.16257 -0.017506 -0.02728 rpy=1.5703 0 2.4131 -> xyz=-0.016997 -0.12029 0.12064 rpy=0 0 0
- joint 2A_joint: origin xyz=-0.36753 -1.0213 -0.20467 rpy=1.5708 0 0 -> xyz=-0.12585 0.0044155 0.03165 rpy=0 0 -0.54114
- joint 2B_joint: axis 0.032866 0.05873 -0.99773 -> -0.48474 0.87466 0; origin xyz=-0.068306 -0.032169 -0.0035499 rpy=-1.5708 -1.0606 -2.7029 -> xyz=-0.066596 -0.035591 -0.0026987 rpy=0 0 0
- joint 2C_joint: axis 0 1 0 -> -0.48474 0.87466 0; origin xyz=0.16412 0.045526 0.022943 rpy=-1.5708 -0.067352 1.0606 -> xyz=-0.10904 -0.052825 0.121 rpy=0 0 0
- joint 3A_joint: origin xyz=-0.36532 -1.0213 -0.07879 rpy=1.5708 0 0 -> xyz=-0.059099 0.11119 0.03165 rpy=0 0 -0.54114
- joint 3B_joint: axis -0.051301 -0.1164 -0.99188 -> 0.69644 0.71761 0; origin xyz=-0.060496 0.045175 -0.0035497 rpy=-1.5708 -1.1557 2.4987 -> xyz=-0.053387 0.0534 -0.0026985 rpy=0 0 0
- joint 3C_joint: axis 0 -1 0.00011568 -> 0.69644 0.71761 0; origin xyz=0.16875 0.027774 -0.011985 rpy=1.4434 0 -0.41512 -> xyz=-0.062549 0.069952 0.14324 rpy=0 0 0
- joint 4A_joint: origin xyz=-0.2552 -1.0213 -0.017762 rpy=1.5708 0 0 -> xyz=0.066747 0.10678 0.03165 rpy=0 0 -0.54114
- joint 4B_joint: axis -0.049746 -0.13238 -0.98995 -> 0.9964 -0.084827 0; origin xyz=-0.004393 0.075374 -0.0035497 rpy=-1.5708 -1.2114 1.6278 -> xyz=0.007552 0.075132 -0.0026985 rpy=0 0 0
- joint 4C_joint: axis 0 -1 6.0305E-05 -> 0.9964 -0.084827 0; origin xyz=0.15545 0.070709 -0.017273 rpy=1.429 0 -0.35944 -> xyz=0.016913 0.12032 0.12066 rpy=0 0 0
- joint 5A_joint: origin xyz=-0.14729 -1.0213 -0.082616 rpy=1.5708 0 0 -> xyz=0.12585 -0.0044158 0.03165 rpy=0 0 -0.54114
- joint 5B_joint: axis 0.010235 0.031305 -0.99946 -> 0.42519 -0.9051 0; origin xyz=0.069335 0.029885 -0.0035501 rpy=-1.5708 -1.2548 0.40578 -> xyz=0.068828 0.031058 -0.0026988 rpy=0 0 0
- joint 5C_joint: axis 0 0 0 -> 0.42519 -0.9051 0; origin xyz=0.1527 0.078405 -0.020579 rpy=1.603 -0.0070889 -0.099179 -> xyz=0.086185 -0.27621 0.1203 rpy=0 0 0
- joint 6A_joint: origin xyz=-0.1495 -1.0213 -0.2085 rpy=1.5708 0 0 -> xyz=0.059099 -0.11119 0.03165 rpy=0 0 -0.54114
- joint 6B_joint: axis -0.032178 0.99947 -0.0046377 -> -0.57232 -0.82003 0; origin xyz=0.070372 -0.031996 -0.003549 rpy=0 0.1431 2.4997 -> xyz=0.061253 -0.044157 -0.0026991 rpy=0 0 0
- joint 6C_joint: axis 0 0 0 -> -0.57232 -0.82003 0; origin xyz=-0.13678 0.037162 0.090718 rpy=0.032483 -1.4277 3.1416 -> xyz=0.12229 0.24662 0.1208 rpy=0 0 0

Commit message: Correción de ejes en la pata 5y6 link C

File: hexapod_description/urdf/hexapod_description.urdf (robot description, URDF)
Before this commit: robot hexapod_description, 19 links, 18 joints
Links:
- link 1C_link: mass 0.0544820458081967 -> 0.0544820458081966
- link 3A_link: mass 0.0263699508271746 -> 0.0263699508271745
- link 3C_link: mass 0.0544820458081965 -> 0.0544820458081966
- link 4B_link: mass 0.0393326464251387 -> 0.0393326464251386
- link 5C_link: mass 0.0544820458081965 -> 0.0544820458081964
- link 6C_link: mass 0.0544820458081965 -> 0.054482
Joints:
- joint 1A_joint: axis 0 0 0.999999999991391 -> 0 0 1; origin xyz=-0.0667468494517693 -0.106777799204074 0.0316495863697956 rpy=0 0 -0.541135476375613 -> xyz=-0.066747 -0.10678 0.03165 rpy=0 0 -0.54114
- joint 1B_joint: axis -0.99634 0.085496 0 -> -0.996338495646665 0.0854962109391992 0; origin xyz=-0.0076049 -0.075127 -0.002699 rpy=0 0 0 -> xyz=-0.00760490724250368 -0.0751266443986717 -0.00269900311088156 rpy=0 0 0
- joint 2B_joint: axis -0.48474 0.87466 0 -> -0.484736668052907 0.874660141213748 0; origin xyz=-0.066596 -0.035591 -0.0026987 rpy=0 0 0 -> xyz=-0.0665963742689142 -0.0355912800079509 -0.00269872535340721 rpy=0 0 0
- joint 3B_joint: axis 0.69644 0.71761 0 -> 0.696443909967172 0.717611231983724 0; origin xyz=-0.053387 0.0534 -0.0026985 rpy=0 0 0 -> xyz=-0.0533873782981206 0.0533996389354673 -0.00269846185166944 rpy=0 0 0
- joint 4B_joint: axis 0.9964 -0.084827 0 -> 0.996395716648548 -0.0848267401051073 0; origin xyz=0.007552 0.075132 -0.0026985 rpy=0 0 0 -> xyz=0.00755197903724675 0.0751319969361967 -0.00269854049076024 rpy=0 0 0
- joint 5B_joint: axis 0.42519 -0.9051 0 -> 0.425192570892761 -0.905102909972711 0; origin xyz=0.068828 0.031058 -0.0026988 rpy=0 0 0 -> xyz=0.0688275229088763 0.0310583245155329 -0.00269883901400592 rpy=0 0 0
- joint 5C_joint: origin xyz=0.086185 -0.27621 0.1203 rpy=0 0 0 -> xyz=0.11251 0.045505 0.1208 rpy=0 0 0
- joint 6A_joint: axis 0 0 1 -> 0 0 0.999999999991391; origin xyz=0.059099 -0.11119 0.03165 rpy=0 0 -0.54114 -> xyz=0.0590987552322091 -0.111193443404212 0.0316495166771902 rpy=0 0 -0.541135476375613
- joint 6B_joint: axis -0.57232 -0.82003 0 -> -0.572319986773635 -0.820030385252709 0; origin xyz=0.061253 -0.044157 -0.0026991 rpy=0 0 0 -> xyz=0.0612532738303673 -0.0441574849800916 -0.0026990706223573 rpy=0 0 0
- joint 6C_joint: origin xyz=0.12229 0.24662 0.1208 rpy=0 0 0 -> xyz=0.095967 -0.075088 0.1203 rpy=0 0 0

Commit message: ACTUALIZACION SIST COORD EN SOLIDWORKS

File: hexapod_description/urdf/hexapod_description.urdf (robot description, URDF)
Before this commit: robot hexapod_description, 19 links, 18 joints
Links:
- link 1A_link: mass 0.0263699506965419 -> 0.0263699506975587
- link 1B_link: mass 0.0393326464255896 -> 0.0393326464265752
- link 1C_link: mass 0.0544820458081966 -> 0.0544820458081965
- link 2B_link: mass 0.0393326465544564 -> 0.0393326465544565
- link 3A_link: mass 0.0263699508271745 -> 0.0263699508271746
- link 3B_link: mass 0.0393326465562273 -> 0.0393326465562279
- link 4A_link: mass 0.0263699506960721 -> 0.0263699506961657
- link 4B_link: mass 0.0393326464251386 -> 0.0393326464252295
- link 5A_link: mass 0.0263699506893305 -> 0.0263699506895398
- link 5B_link: mass 0.0393326465545736 -> 0.0393326465545709
- link 5C_link: mass 0.0544820458081964 -> 0.0544820458081966
- link 6A_link: mass 0.0263699508281301 -> 0.02636995082813
- link 6B_link: mass 0.0393326465581178 -> 0.0393326465581168
- link 6C_link: mass 0.054482 -> 0.0544820458081965
Joints:
- joint 1A_joint: axis 0 0 1 -> 0 0.000189825421871335 0.999999981983154; origin xyz=-0.066747 -0.10678 0.03165 rpy=0 0 -0.54114 -> xyz=-0.0667468494517693 -0.106777799204074 0.0316495863697956 rpy=0.000187289878885293 0 -2.12946850394786
- joint 1B_joint: axis -0.996338495646665 0.0854962109391992 0 -> -0.0695536721571611 -0.997578192840082 0.000189365704729826; origin xyz=-0.00760490724250368 -0.0751266443986717 -0.00269900311088156 rpy=0 0 0 -> xyz=0.0752386562540257 -0.00640318117526778 -0.00269755643730618 rpy=0 0 0
- joint 1C_joint: axis -0.99634 0.085496 0 -> -0.0695536721571234 -0.997578192840085 0.000189365704778719; origin xyz=-0.016997 -0.12029 0.12064 rpy=0 0 0 -> xyz=0.120546165521457 -0.015048025350051 0.120647727640648 rpy=0 0 0
- joint 2A_joint: axis 0 0 1 -> 0 0 0.999999999992758; origin xyz=-0.12585 0.0044155 0.03165 rpy=0 0 -0.54114 -> xyz=-0.125845591742144 0.00441551350601397 0.0316500696923352 rpy=0 0 3.10651925204043
- joint 2B_joint: axis -0.484736668052907 0.874660141213748 0 -> 0 -0.999999999992758 0; origin xyz=-0.0665963742689142 -0.0355912800079509 -0.00269872535340721 rpy=0 0 0 -> xyz=0.0755015911121684 -0.00115142974218954 -0.00269876749323283 rpy=0 0 0
- joint 2C_joint: axis -0.48474 0.87466 0 -> 0 -0.999999999992758 0; origin xyz=-0.10904 -0.052825 0.121 rpy=0 0 0 -> xyz=0.12097495075034 -0.00664953949368554 0.121002671452846 rpy=0 0 0
- joint 3A_joint: axis 0 0 1 -> 0 0 0.999999999992459; origin xyz=-0.059099 0.11119 0.03165 rpy=0 0 -0.54114 -> xyz=-0.0590987293485508 0.111193182015965 0.0316504833222655 rpy=0 0 2.05932170084572
- joint 3B_joint: axis 0.696443909967172 0.717611231983724 0 -> -0.227149790678758 -0.973859832101259 0; origin xyz=-0.0533873782981206 0.0533996389354673 -0.00269846185166944 rpy=0 0 0 -> xyz=0.0732672863787103 -0.0182657395441897 -0.00269870093818958 rpy=0 0 0
- joint 3C_joint: axis 0.69644 0.71761 0 -> -0.227149790678759 -0.973859832101259 0; origin xyz=-0.062549 0.069952 0.14324 rpy=0 0 0 -> xyz=0.0896470917080924 -0.027733299889676 0.143235135491589 rpy=0 0 0
- joint 4A_joint: axis 0 0 1 -> 0 -0.000189825421852773 0.999999981983154; origin xyz=0.066747 0.10678 0.03165 rpy=0 0 -0.54114 -> xyz=0.0667468753354276 0.106777537815826 0.0316504136296591 rpy=-0.000187289878885293 0 1.01212414964193
- joint 4B_joint: axis 0.996395716648548 -0.0848267401051073 0 -> -0.067341098883768 -0.99772999380135 -0.000189394520411146; origin xyz=0.00755197903724675 0.0751319969361967 -0.00269854049076024 rpy=0 0 0 -> xyz=0.0752519835596818 -0.00624345785823413 -0.00269995709093918 rpy=0 0 0
- joint 4C_joint: axis 0.9964 -0.084827 0 -> -0.0673410988837552 -0.997729993801351 -0.000189394520251638; origin xyz=0.016913 0.12032 0.12066 rpy=0 0 0 -> xyz=0.120591722612344 -0.0148405749057716 0.120657273965076 rpy=0 0 0
- joint 5A_joint: axis 0 0 1 -> 0 0 0.999999999992758; origin xyz=0.12585 -0.0044158 0.03165 rpy=0 0 -0.54114 -> xyz=0.125845617625808 -0.00441577489426207 0.0316499303071216 rpy=0 0 -0.0350734015493665
- joint 5B_joint: axis 0.425192570892761 -0.905102909972711 0 -> -0.0658773160112557 -0.997827730232395 0; origin xyz=0.0688275229088763 0.0310583245155329 -0.00269883901400592 rpy=0 0 0 -> xyz=0.0752608794529679 -0.00613572763718961 -0.00269879522635974 rpy=0 0 0
- joint 5C_joint: axis 0.42519 -0.9051 0 -> -0.0658773160112644 -0.997827730232394 0; origin xyz=0.11251 0.045505 0.1208 rpy=0 0 0 -> xyz=0.120466525966111 -0.0146350482342145 0.120807379890955 rpy=0 0 0
- joint 6A_joint: axis 0 0 0.999999999991391 -> 0 0 0.999999999992459; origin xyz=0.0590987552322091 -0.111193443404212 0.0316495166771902 rpy=0 0 -0.541135476375613 -> xyz=0.0590987552322091 -0.111193443404212 0.0316495166771902 rpy=0 0 -1.08227095274408
- joint 6B_joint: axis -0.572319986773635 -0.820030385252709 0 -> -0.0681438930759001 -0.997675503268196 0; origin xyz=0.0612532738303673 -0.0441574849800916 -0.0026990706223573 rpy=0 0 0 -> xyz=0.0752472515487932 -0.00630076885737318 -0.00269879634505443 rpy=0 0 0
- joint 6C_joint: axis -0.57232 -0.82003 0 -> -0.068143893075898 -0.997675503268196 0; origin xyz=0.095967 -0.075088 0.1203 rpy=0 0 0 -> xyz=0.120933977901671 -0.0149333124138473 0.120302680099782 rpy=0 0 0

Commit message: INTENTO NUEVO SOLIDWORKS CON SISTEMAS P

File: hexapod_description/urdf/hexapod_description.urdf (robot description, URDF)
Before this commit: robot hexapod_description, 19 links, 18 joints
Links:
- added link 1P_link, mass 0.065522052028268; collision mesh filename=package://hexapod_description/meshes/1P_link.STL; visual mesh filename=package://hexapod_description/meshes/1P_link.STL
- added link 2P_link, mass 0.0655220520282681; collision mesh filename=package://hexapod_description/meshes/2P_link.STL; visual mesh filename=package://hexapod_description/meshes/2P_link.STL
- added link 3P_link, mass 0.0655220520282678; collision mesh filename=package://hexapod_description/meshes/3P_link.STL; visual mesh filename=package://hexapod_description/meshes/3P_link.STL
- added link 4P_link, mass 0.065522052028268; collision mesh filename=package://hexapod_description/meshes/4P_link.STL; visual mesh filename=package://hexapod_description/meshes/4P_link.STL
- added link 5P_link, mass 0.065522052028268; collision mesh filename=package://hexapod_description/meshes/5P_link.STL; visual mesh filename=package://hexapod_description/meshes/5P_link.STL
- added link 6P_link, mass 0.065522052028268; collision mesh filename=package://hexapod_description/meshes/6P_link.STL; visual mesh filename=package://hexapod_description/meshes/6P_link.STL
- link 1A_link: mass 0.0263699506975587 -> 0.0329624380889454
- link 1B_link: mass 0.0393326464265752 -> 0.0491658077507467
- link 1C_link: mass 0.0544820458081965 -> 0.0681025572602457
- link 2A_link: mass 0.0263699508381414 -> 0.0329624385476769
- link 2B_link: mass 0.0393326465544565 -> 0.0491658081930703
- link 2C_link: mass 0.0544820458081966 -> 0.068102557260246
- link 3A_link: mass 0.0263699508271746 -> 0.0329624385357417
- link 3B_link: mass 0.0393326465562279 -> 0.0491658081987106
- link 3C_link: mass 0.0544820458081966 -> 0.0681025572602457
- link 4A_link: mass 0.0263699506961657 -> 0.0329624380888626
- link 4B_link: mass 0.0393326464252295 -> 0.049165807750671
- link 4C_link: mass 0.0544820458081966 -> 0.0681025572602458
- link 5A_link: mass 0.0263699506895398 -> 0.0329624385477412
- link 5B_link: mass 0.0393326465545709 -> 0.0491658081930705
- link 5C_link: mass 0.0544820458081966 -> 0.0681025572602457
- link 6A_link: mass 0.02636995082813 -> 0.0329624385357485
- link 6B_link: mass 0.0393326465581168 -> 0.0491658081987123
- link 6C_link: mass 0.0544820458081965 -> 0.0681025572602456
- link base_link: mass 0.406550708950941 -> 0.508188386188677
Joints:
- added joint 1P_joint: type fixed, parent 1C_link, child 1P_link, origin xyz=0.11638 -0.00085 0 rpy=0 0.30547 0, axis 0 0 0, limit lower=-1 upper=1 effort=0 velocity=0
- added joint 2P_joint: type fixed, parent 2C_link, child 2P_link, origin xyz=0.11639 -0.00085 0 rpy=0 0.30533 0, axis 0 0 0, limit lower=-1 upper=1 effort=0 velocity=0
- added joint 3P_joint: type fixed, parent 3C_link, child 3P_link, origin xyz=0.11639 -0.00085 0 rpy=0 0.30533 0, axis 0 0 0, limit lower=-1 upper=1 effort=0 velocity=0
- added joint 4P_joint: type fixed, parent 4C_link, child 4P_link, origin xyz=0.11639 -0.00085 0 rpy=0 0.30533 0, axis 0 0 0, limit lower=-1 upper=1 effort=0 velocity=0
- added joint 5P_joint: type fixed, parent 5C_link, child 5P_link, origin xyz=0.11639 -0.00085 0 rpy=0 0.30533 0, axis 0 0 0, limit lower=-1 upper=1 effort=0 velocity=0
- added joint 6P_joint: type fixed, parent 6C_link, child 6P_link, origin xyz=0.11639 -0.00085 0 rpy=0 0.30533 0, axis 0 0 0, limit lower=-1 upper=1 effort=0 velocity=0
- joint 1A_joint: axis 0 0.000189825421871335 0.999999981983154 -> -0.035728 0 0.99936; limit lower=0 upper=0 effort=0 velocity=0 -> lower=-1 upper=1 effort=0 velocity=0; origin xyz=-0.0667468494517693 -0.106777799204074 0.0316495863697956 rpy=0.000187289878885293 0 -2.12946850394786 -> xyz=-0.066747 -0.10678 0.03165 rpy=0 0.035739 -2.1204
- joint 1B_joint: axis -0.0695536721571611 -0.997578192840082 0.000189365704729826 -> 0 -1 0; limit lower=0 upper=0 effort=0 velocity=0 -> lower=-1 upper=1 effort=0 velocity=0; origin xyz=0.0752386562540257 -0.00640318117526778 -0.00269755643730618 rpy=0 0 0 -> xyz=0.075536 -0.001836 0 rpy=0.00047569 -0.82122 -0.0094139
- joint 1C_joint: axis -0.0695536721571234 -0.997578192840085 0.000189365704778719 -> 0 -1 0; limit lower=0 upper=0 effort=0 velocity=0 -> lower=-1 upper=1 effort=0 velocity=0; origin xyz=0.120546165521457 -0.015048025350051 0.120647727640648 rpy=0 0 0 -> xyz=0.17108 -0.00665 0 rpy=3.1416 1.0908 3.1416
- joint 2A_joint: axis 0 0 0.999999999992758 -> 0 0 1; limit lower=0 upper=0 effort=0 velocity=0 -> lower=-1 upper=1 effort=0 velocity=0; origin xyz=-0.125845591742144 0.00441551350601397 0.0316500696923352 rpy=0 0 3.10651925204043 -> xyz=-0.12582 0.0044184 0.01135 rpy=0 0 -3.0654; type revolute -> continuous
- joint 2B_joint: axis 0 -0.999999999992758 0 -> 0 -1 0; limit lower=0 upper=0 effort=0 velocity=0 -> lower=-1 upper=1 effort=0 velocity=0; origin xyz=0.0755015911121684 -0.00115142974218954 -0.00269876749323283 rpy=0 0 0 -> xyz=0.074928 -0.009527 0.017601 rpy=0 -0.78551 -0.11127
- joint 2C_joint: axis 0 -0.999999999992758 0 -> 0 -1 0; limit lower=0 upper=0 effort=0 velocity=0 -> lower=-1 upper=1 effort=0 velocity=0; origin xyz=0.12097495075034 -0.00664953949368554 0.121002671452846 rpy=0 0 0 -> xyz=0.1711 -0.00665 0 rpy=-3.1416 1.0906 -3.1416
- joint 3A_joint: axis 0 0 0.999999999992459 -> -0.035728 0 0.99936; limit lower=0 upper=0 effort=0 velocity=0 -> lower=-1 upper=1 effort=0 velocity=0; origin xyz=-0.0590987293485508 0.111193182015965 0.0316504833222655 rpy=0 0 2.05932170084572 -> xyz=-0.059099 0.11119 0.03165 rpy=0 0.035732 2.0683
- joint 3B_joint: axis -0.227149790678758 -0.973859832101259 0 -> 5.4838E-05 -1 -5.485E-05; limit lower=0 upper=0 effort=0 velocity=0 -> lower=-1 upper=1 effort=0 velocity=0; origin xyz=0.0732672863787103 -0.0182657395441897 -0.00269870093818958 rpy=0 0 0 -> xyz=0.075536 -0.001836 0 rpy=0.0004757 -0.82124 -0.0094139
- joint 3C_joint: axis -0.227149790678759 -0.973859832101259 0 -> 2.3315E-05 -1 7.3974E-05; limit lower=0 upper=0 effort=0 velocity=0 -> lower=-1 upper=1 effort=0 velocity=0; origin xyz=0.0896470917080924 -0.027733299889676 0.143235135491589 rpy=0 0 0 -> xyz=0.1711 -0.00665 0 rpy=3.1416 1.0906 3.1416
- joint 4A_joint: axis 0 -0.000189825421852773 0.999999981983154 -> -0.035728 0 0.99936; limit lower=0 upper=0 effort=0 velocity=0 -> lower=-1 upper=1 effort=0 velocity=0; origin xyz=0.0667468753354276 0.106777537815826 0.0316504136296591 rpy=-0.000187289878885293 0 1.01212414964193 -> xyz=0.066747 0.10678 0.03165 rpy=0 0.035732 1.0212
- joint 4B_joint: axis -0.067341098883768 -0.99772999380135 -0.000189394520411146 -> -3.1787E-05 -1 3.1795E-05; limit lower=0 upper=0 effort=0 velocity=0 -> lower=-1 upper=1 effort=0 velocity=0; origin xyz=0.0752519835596818 -0.00624345785823413 -0.00269995709093918 rpy=0 0 0 -> xyz=0.075536 -0.001836 0 rpy=0.00047571 -0.82125 -0.0094139
- joint 4C_joint: axis -0.0673410988837552 -0.997729993801351 -0.000189394520251638 -> -1.3515E-05 -1 -4.288E-05; limit lower=0 upper=0 effort=0 velocity=0 -> lower=-1 upper=1 effort=0 velocity=0; origin xyz=0.120591722612344 -0.0148405749057716 0.120657273965076 rpy=0 0 0 -> xyz=0.1711 -0.00665 0 rpy=-3.1416 1.0906 -3.1416
- joint 5A_joint: axis 0 0 0.999999999992758 -> -0.035728 0 0.99936; limit lower=0 upper=0 effort=0 velocity=0 -> lower=-1 upper=1 effort=0 velocity=0; origin xyz=0.125845617625808 -0.00441577489426207 0.0316499303071216 rpy=0 0 -0.0350734015493665 -> xyz=0.12585 -0.0044158 0.03165 rpy=0 0.035736 -0.026443
- joint 5B_joint: axis -0.0658773160112557 -0.997827730232395 0 -> 0 -1 0; limit lower=0 upper=0 effort=0 velocity=0 -> lower=-1 upper=1 effort=0 velocity=0; origin xyz=0.0752608794529679 -0.00613572763718961 -0.00269879522635974 rpy=0 0 0 -> xyz=0.075536 -0.001836 0 rpy=0.00047569 -0.82121 -0.0094139
- joint 5C_joint: axis -0.0658773160112644 -0.997827730232394 0 -> 0 -1 0; limit lower=0 upper=0 effort=0 velocity=0 -> lower=-1 upper=1 effort=0 velocity=0; origin xyz=0.120466525966111 -0.0146350482342145 0.120807379890955 rpy=0 0 0 -> xyz=0.1711 -0.00665 0 rpy=3.1416 1.0907 3.1416
- joint 6A_joint: axis 0 0 0.999999999992459 -> -0.035728 0 0.99936; limit lower=0 upper=0 effort=0 velocity=0 -> lower=-1 upper=1 effort=0 velocity=0; origin xyz=0.0590987552322091 -0.111193443404212 0.0316495166771902 rpy=0 0 -1.08227095274408 -> xyz=0.059099 -0.11119 0.03165 rpy=0 0.03574 -1.0732
- joint 6B_joint: axis -0.0681438930759001 -0.997675503268196 0 -> 0 -1 0; limit lower=0 upper=0 effort=0 velocity=0 -> lower=-1 upper=1 effort=0 velocity=0; origin xyz=0.0752472515487932 -0.00630076885737318 -0.00269879634505443 rpy=0 0 0 -> xyz=0.075536 -0.001836 0 rpy=0.00047571 -0.82125 -0.0094139
- joint 6C_joint: axis -0.068143893075898 -0.997675503268196 0 -> 0 -1 0; limit lower=0 upper=0 effort=0 velocity=0 -> lower=-1 upper=1 effort=0 velocity=0; origin xyz=0.120933977901671 -0.0149333124138473 0.120302680099782 rpy=0 0 0 -> xyz=0.1711 -0.00665 0 rpy=-3.1416 1.0906 3.1416
